File: UniESP.kicad_sch (KiCad schematic)
At the start: 58 parts, among them J1 Power Conn, J2 12V Input, J3 RTC conn, J4 Extra conn, J5 Motor2_Output, J6 M2_out, J7 Motor1_Output, J8 M1_out, U1 TPS5430DDA, U2 ESP32-DevKitV1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

Commit message: Added PEC filtering
Connections:
- net +12V: now also J1.2 (Pin_2)
- net +3V3: no longer J1.3 (Pin_3)
- net +5V: now also J1.3 (Pin_3)
- net GND: now also J4.1 (Pin_1), J4.2 (Pin_2); no longer J1.2 (Pin_2)
Changed lines of the file:
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@@
 	(paper "A4")
 	(junction
-		(at 19.05 88.9)
+		(at 186.69 54.61)
 		(diameter 0)
 		(color 0 0 0 0)
 	)
 	(junction
-		(at 186.69 54.61)
+		(at 190.5 29.21)
 		(diameter 0)
 		(color 0 0 0 0)
 	)
 	(junction
-		(at 190.5 29.21)
+		(at 77.47 49.53)
 		(diameter 0)
 		(color 0 0 0 0)
@@
 	)
 	(junction
-		(at 19.05 96.52)
-		(diameter 0)
-		(color 0 0 0 0)
-	)
-	(junction
 		(at 46.99 173.99)
 		(diameter 0)
@@
 	(wire
 		(pts
+			(xy 77.47 46.99) (xy 77.47 49.53)
+		)
+		(stroke
+			(width 0)
+			(type default)
+		)
+	)
+	(wire
+		(pts
 			(xy 46.99 119.38) (xy 48.26 119.38)
 		)
@@
 	(wire
 		(pts
+			(xy 77.47 49.53) (xy 77.47 52.07)
+		)
+		(stroke
+			(width 0)
+			(type default)
+		)
+	)
+	(wire
+		(pts
 			(xy 46.99 176.53) (xy 46.99 173.99)
 		)
@@
 	(wire
 		(pts
-			(xy 19.05 93.98) (xy 19.05 96.52)
-		)
-		(stroke
-			(width 0)
-			(type default)
-		)
-	)
-	(wire
-		(pts
-			(xy 19.05 88.9) (xy 19.05 91.44)
-		)
-		(stroke
-			(width 0)
-			(type default)
-		)
-	)
-	(wire
-		(pts
 			(xy 200.66 134.62) (xy 186.69 134.62)
 		)
@@
 	)
 	(symbol
+		(lib_id "power:+12V")
+		(at 19.05 93.98 90)
+		(unit 1)
+		(exclude_from_sim no)
+		(in_bom yes)
+		(on_board yes)
+		(dnp no)
+		(fields_autoplaced yes)
+		(property "Reference" "#PWR046"
+			(at 22.86 93.98 0)
+			(effects
+				(font
+					(size 1.27 1.27)
+				)
+				(hide yes)
+			)
+		)
+		(property "Value" "+12V"
+			(at 13.97 93.98 0)
+			(effects
+				(font
+					(size 1.27 1.27)
+				)
+			)
+		)
+		(property "Footprint" ""
+			(at 19.05 93.98 0)
+			(effects
+				(font
+					(size 1.27 1.27)
+				)
+				(hide yes)
+			)
+		)
+		(property "Datasheet" ""
+			(at 19.05 93.98 0)
+			(effects
+				(font
+					(size 1.27 1.27)
+				)
+				(hide yes)
+			)
+		)
+		(property "Description" "Power symbol creates a global label with name \"+12V\""
+			(at 19.05 93.98 0)
+			(effects
+				(font
+					(size 1.27 1.27)
+				)
+				(hide yes)
+			)
+		)
+		(pin "1"
+		)
+		(instances
+			(project "UniESP"
+				(path "/5d3f246f-f73d-440c-84ab-058d6ba53936"
+					(reference "#PWR046")
+					(unit 1)
+				)
+			)
+		)
+	)
+	(symbol
 		(lib_id "Device:R")
 		(at 146.05 167.64 90)
@@
 	)
 	(symbol
+		(lib_id "power:+5V")
+		(at 19.05 91.44 90)
+		(unit 1)
+		(exclude_from_sim no)
+		(in_bom yes)
+		(on_board yes)
+		(dnp no)
+		(fields_autoplaced yes)
+		(property "Reference" "#PWR045"
+			(at 22.86 91.44 0)
+			(effects
+				(font
+					(size 1.27 1.27)
+				)
+				(hide yes)
+			)
+		)
+		(property "Value" "+5V"
+			(at 15.24 91.4399 90)
+			(effects
+				(font
+					(size 1.27 1.27)
+				)
+				(justify left)
+			)
+		)
+		(property "Footprint" ""
+			(at 19.05 91.44 0)
+			(effects
+				(font
+					(size 1.27 1.27)
+				)
+				(hide yes)
+			)
+		)
+		(property "Datasheet" ""
+			(at 19.05 91.44 0)
+			(effects
+				(font
+					(size 1.27 1.27)
+				)
+				(hide yes)
+			)
+		)
+		(property "Description" "Power symbol creates a global label with name \"+5V\""
+			(at 19.05 91.44 0)
+			(effects
+				(font
+					(size 1.27 1.27)
+				)
+				(hide yes)
+			)
+		)
+		(pin "1"
+		)
+		(instances
+			(project "UniESP"
+				(path "/5d3f246f-f73d-440c-84ab-058d6ba53936"
+					(reference "#PWR045")
+					(unit 1)
+				)
+			)
+		)
+	)
+	(symbol
 		(lib_id "CUSTOM:ESP32-DevKitV1")
 		(at 50.8 54.61 0)
@@
 					(unit 1)
 				)
+			)
+		)
+	)
+	(symbol
+		(lib_id "power:GND")
+		(at 77.47 52.07 0)
+		(unit 1)
+		(exclude_from_sim no)
+		(in_bom yes)
+		(on_board yes)
+		(dnp no)
+		(fields_autoplaced yes)
+		(property "Reference" "#PWR047"
+			(at 77.47 58.42 0)
+			(effects
+				(font
+					(size 1.27 1.27)
+				)
+				(hide yes)
+			)
+		)
+		(property "Value" "GND"
+			(at 77.47 57.15 0)
+			(effects
+				(font
+					(size 1.27 1.27)
+				)
+			)
+		)
+		(property "Footprint" ""
+			(at 77.47 52.07 0)
+			(effects
+				(font
+					(size 1.27 1.27)
+				)
+				(hide yes)
+			)
+		)
+		(property "Datasheet" ""
+			(at 77.47 52.07 0)
+			(effects
+				(font
+					(size 1.27 1.27)
+				)
+				(hide yes)
+			)
+		)
+		(property "Description" "Power symbol creates a global label with name \"GND\" , ground"
+			(at 77.47 52.07 0)
+			(effects
+				(font
+					(size 1.27 1.27)
+				)
+				(hide yes)
+			)
+		)
+		(pin "1"
+		)
+		(instances
+			(project "UniESP"
+				(path "/5d3f246f-f73d-440c-84ab-058d6ba53936"
+					(reference "#PWR047")
+					(unit 1)
+				)
